File: electronics/trezor_v1.1_usb_c/trezor_v1.1.kicad_pcb (KiCad board)
At the start: 16 copper layers, 50 x 26.7 mm, 34 parts, among them IC1 MCP1703T-3302E/CB, J1 USB_C_Receptacle_USB2.0, K2 SWD, Q2 8MHz, U1 STM32F205RET6, U3 DISPLAY

Commit message: Minor silkscreen fixes, add specifier for JLC order number
Other:
- copper layers 16 -> 2
- board text added: "JLCJLCJLCJLC"
- board text removed: "BOT"
- board text removed: "TOP"
Changed lines of the file:
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@@
   (general
     (thickness 1.6)
-    (drawings 216)
+    (drawings 215)
     (tracks 598)
     (zones 0)
@@
   (page A4)
   (layers
-    (0 Top signal hide)
-    (1 Route2 signal hide)
-    (2 Route3 signal hide)
-    (3 Route4 signal hide)
-    (4 Route5 signal hide)
-    (5 Route6 signal hide)
-    (6 Route7 signal hide)
-    (7 Route8 signal hide)
-    (8 Route9 signal hide)
-    (9 Route10 signal hide)
-    (10 Route11 signal hide)
-    (11 Route12 signal hide)
-    (12 Route13 signal hide)
-    (13 Route14 signal hide)
-    (14 Route15 signal hide)
-    (31 Bottom signal hide)
-    (32 B.Adhes user hide)
-    (33 F.Adhes user hide)
-    (34 B.Paste user hide)
-    (35 F.Paste user hide)
+    (0 Top signal)
+    (31 Bottom signal)
+    (32 B.Adhes user)
+    (33 F.Adhes user)
+    (34 B.Paste user)
+    (35 F.Paste user)
     (36 B.SilkS user)
     (37 F.SilkS user)
-    (38 B.Mask user hide)
-    (39 F.Mask user hide)
-    (40 Dwgs.User user hide)
-    (41 Cmts.User user hide)
-    (42 Eco1.User user hide)
-    (43 Eco2.User user hide)
+    (38 B.Mask user)
+    (39 F.Mask user)
+    (40 Dwgs.User user)
+    (41 Cmts.User user)
+    (42 Eco1.User user)
+    (43 Eco2.User user)
     (44 Edge.Cuts user)
-    (45 Margin user hide)
-    (46 B.CrtYd user hide)
-    (47 F.CrtYd user hide)
-    (48 B.Fab user hide)
-    (49 F.Fab user hide)
+    (45 Margin user)
+    (46 B.CrtYd user)
+    (47 F.CrtYd user)
+    (48 B.Fab user)
+    (49 F.Fab user)
   )
   (setup
@@
       (plotinvisibletext false)
       (padsonsilk false)
-      (subtractmaskfromsilk false)
+      (subtractmaskfromsilk true)
       (outputformat 1)
       (mirror false)
-      (drillshape 1)
+      (drillshape 0)
       (scaleselection 1)
-      (outputdirectory ""))
+      (outputdirectory "export/"))
   )
   (net 0 "")
@@
   (module trezor_v1.1:0402 (layer Top)
     (at 138.3284 95.1992 180)
-    (fp_text reference C8 (at 2.5654 -0.5588 180) (layer F.SilkS)
+    (fp_text reference C8 (at 2.8829 -0.5588 180) (layer F.SilkS)
       (effects (font (size 1 1) (thickness 0.15)) (justify left bottom))
     )
@@
   (module trezor_v1.1:0402 (layer Top)
     (at 141.478 110.4392)
-    (fp_text reference C9 (at -2.7305 0.5588) (layer F.SilkS)
+    (fp_text reference C9 (at -2.8575 0.4953) (layer F.SilkS)
       (effects (font (size 1 1) (thickness 0.15)) (justify left bottom))
     )
@@
   (module trezor_v1.1:0402 (layer Top)
     (at 144.2212 108.4072 180)
-    (fp_text reference C13 (at 2.2352 -1.5748) (layer F.SilkS)
+    (fp_text reference C13 (at 2.2352 -1.7018) (layer F.SilkS)
       (effects (font (size 1 1) (thickness 0.15)) (justify left bottom))
     )
@@
     (pad 1 smd rect (at -0.8 0 270) (size 0.8 1) (layers Top F.Paste F.Mask)
       (net 1 GND) (solder_mask_margin 0.1016))
+  )
+  (gr_text JLCJLCJLCJLC (at 169.8625 104.4575 90) (layer B.SilkS)
+    (effects (font (size 0.9 0.9) (thickness 0.15)) (justify mirror))
   )
   (gr_text VDD (at 141.224 93.98 90) (layer B.SilkS)
@@
   (gr_line (start 128.8288 98.4504) (end 129.413 98.4758) (layer Edge.Cuts) (width 0.05))
   (gr_line (start 129.413 98.4758) (end 129.9718 98.2726) (layer Edge.Cuts) (width 0.05))
-  (gr_text TOP (at 151.13 117.5512) (layer Top)
-    (effects (font (size 1.5 1.5) (thickness 0.3)) (justify left bottom))
-  )
-  (gr_text BOT (at 149.606 117.4496) (layer Bottom)
-    (effects (font (size 1.5 1.5) (thickness 0.3)) (justify left bottom mirror))
-  )
   (gr_line (start 145.6436 108.4072) (end 149.5044 108.4072) (layer Dwgs.User) (width 0.15))
   (gr_line (start 149.5044 108.4072) (end 149.5044 107.4928) (layer Dwgs.User) (width 0.15))

Commit message: Fix solder mask on all footprints, minor trace cleanup
Routing:
- net GND: track 200.9 -> 199.0 mm
Other:
- rule pad_to_mask_clearance: 0.051 -> 0.05
- rule solder_mask_min_width: 0.25 -> 0.05
